File: dobot_circuite/dobot_circuite.sch (KiCad schematic (older format))
At the start: 29 parts, among them J1 USB_A, J2 USB_A, J3 USB_A, J4 USB_A, J5 USB_A, J6 USB_A, J7 HDMI, J8 Jack-DC, J9 HDMI, U1 FE1.1s, U2 FE1.1s, U3 usb_connector, U4 XH_DCJ, U5 usb_connector, U6 HDMI_Hole, U7 HDMI_Hole2, U8 arduino_leonard, Y1 Crystal, Y2 Crystal

Commit message: Add files via upload
Parts:
- removed U2: FE1.1s, hoshina_library:FE1.1s, symbol dobot_circuite-rescue:FE1.1s-hoshina_library-dobot_circuite-rescue-dobot_circui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
- removed U3, U5: usb_connector, hoshina_library:XH4PIN_S, symbol dobot_circuite-rescue:usb_connector-dobot_circuite-cache-dobot_circuite-rescue
- removed U4: XH_DCJ, hoshina_library:S2B-XH-A_DCJ, symbol hoshina_library:XH_DCJ
- removed U6: HDMI_Hole, hoshina_library:HDMI_Hole, symbol hoshina_library:HDMI_Hole
- removed U8: arduino_leonard, hoshina_library:arduino_leonard, symbol hoshina_library:arduino_leonard
- removed Y2: Crystal, hoshina_library:Crystal_SMD_5032-2Pin_5.0x3.2mm, symbol Device:Crystal
- added A1: Arduino_Leonardo_pin_remove_2pin, hoshina_library:arduino_leonard_remove_2pin, symbol hoshina_library:Arduino_Leonardo_pin_remove_2pin
- added D1: LED_green, hoshina_library:LED_1608, symbol Device:LED
- added K1, K2, K3: ALQ105, hoshina_library:ALQ105_akituki, symbol hoshina_library:ALQ105
- added R10, R11, R14, R15, R18, R19, R21, R7: 10k, hoshina_library:register_0603, symbol Device:R
- added R12, R13, R8, R9: 1k/1W, hoshina_library:carbon_register, symbol Device:R
- added R16, R17, R20, R6: 190, hoshina_library:register_0603, symbol Device:R
- added R22: R, hoshina_library:carbon_register, symbol Device:R
- added R23, R24, R29, R30, R31, R32: 5.6k/1w, hoshina_library:carbon_register, symbol Device:R
- added R25, R26, R27, R28: 4.7k, hoshina_library:register_0603, symbol Device:R
- added R3, R4, R5: 5k, hoshina_library:register_0603, symbol Device:R
- added SW1: SW_Push_Dual, hoshina_library:SW_TH_Tactile_Omron_B3F-10xx, symbol Switch:SW_Push_Dual
- added T1, T2, T3: 2SD1781K, hoshina_library:2SD1781, symbol hoshina_library:2SD1781K
- added U10, U12, U13, U14, U15, U17, U18, U19: fhoto_capura_PS817, hoshina_library:fhoto_capra_PS817, symbol hoshina_library:fhoto_capura_PS817
- added U11, U16: terminal_block_4pin_small, hoshina_library:terminal_block_4pin_small, symbol hoshina_library:terminal_block_4pin_small
- added U2, U3, U5: microB_usb_connector, hoshina_library:USB_Micro-B_MC5F-03_aitendo_reverse, symbol hoshina_library:microB_usb_connector
- added U20, U21, U22: diode_GS1010FL, hoshina_library:diode_GS1010FL, symbol hoshina_library:diode_GS1010FL
- added U23, U8: terminal_block_6pin_small, hoshina_library:terminal_block_6pin_small, symbol hoshina_library:terminal_block_6pin_small
- added U9: terminal_block_2pin_small, hoshina_library:terminal_block_2pin_small, symbol hoshina_library:terminal_block_2pin_small
- added hand_electric_line1: hoshina_library_terminal_block_2pin_small, hoshina_library:2pin_power_gnd, symbol dobot_circuite-cache:hoshina_library_terminal_block_2pin_small
- added led1, led10, led11, led2, led3, led4, led5, led6, led7, led8, led9: LED, hoshina_library:LED_1608, symbol hoshina_library:LED
- R2: value R -> 5.6k/1w; footprint hoshina_library:register_0603 -> hoshina_library:carbon_register
Connections:
- net +5V: now also K1.C1, K2.C1, K3.C1, U12.4, U13.4, U14.4, U15.4, U2.5V, U20.1, U21.1, U22.1, U23.6, U3.5V, U5.5V, hand_electric_line1.1
- net GND: now also A1.GND, R25.2, R26.2, R27.2, R28.2, R29.2, R30.2, R31.2, R32.2, SW1.4, T1.E, T2.E, T3.E, U10.2, U12.2, U13.2, U14.2, U15.2, U17.2, U18.2, U19.2, U2.GND, U23.1, U3.GND, U5.GND, hand_electric_line1.2; no longer R2.1
- net at J2.2 (D-): now also U3.D-
- net at J2.3 (D+): now also U3.D+
- net at J4.2 (D-): now also U5.D-
- net at J4.3 (D+): now also U5.D+
- net at U1.DMU: now also U2.D-
- net at U1.DPU: now also U2.D+
- net D13_relay: now reaches R2.2
- net D13_relay: now also K3.NO, U8.1
- new net: A1.RESET, SW1.3
- new net: K1.C2, T1.C, U20.2
- new net: K2.C2, T2.C, U21.2
- new net: K3.C2, T3.C, U22.2
- new net: R3.1, T1.B
- new net: R4.1, T2.B
- new net: R5.1, T3.B
- new net: R6.1, U10.1
- new net: D1.1 (K), R22.1
- new net: R20.1, U19.1
- new net: R17.1, U18.1
- new net: R16.1, U17.1
- new net: R13.1, U15.1
- new net: R12.1, U14.1
- new net: R9.1, U13.1
- new net: R8.1, U12.1
- new net: R2.1, led1.1 (K)
- new net: R23.1, led2.1 (K)
- new net: R24.1, led3.1 (K)
- new net: R29.1, led8.1 (K)
- new net: R30.1, led9.1 (K)
- new net: R31.1, led10.1 (K)
- new net: R32.1, led11.1 (K)
- new net: R25.1, led4.1 (K)
- new net: R26.1, led5.1 (K)
- new net: R27.1, led6.1 (K)
- new net: R28.1, led7.1 (K)
- new net +24V: D1.2 (A), U10.4, U17.4, U18.4, U19.4, U8.2, U8.4, U8.6, U9.2, led1.2 (A), led2.2 (A), led3.2 (A)
- new net A0: A1.A0, U23.5
- new net A1: A1.A1, U23.4
- new net A2: A1.A2, U23.3
- new net A3: A1.A3, U23.2
- new net D10: A1.D10, R6.2
- new net D10_24V: R7.2, U10.3, U11.1, led11.2 (A)
- new net D11: A1.D11, R3.2
- new net D11_relay: K1.NO, R24.2, U8.5
- new net D12: A1.D12, R4.2
- new net D12_relay: K2.NO, R23.2, U8.3
- new net D13: A1.D13, R5.2
- new net D3: A1.D3/SCL, R10.2, U12.3, led5.2 (A)
- new net D3_24V: R8.2, U16.4
- new net D4: A1.D4, R14.2, U14.3, led4.2 (A)
- new net D4_24V: R12.2, U16.3
- new net D5: A1.D5, R11.2, U13.3, led6.2 (A)
- new net D5_24V: R9.2, U16.2
- new net D6: A1.D6, R15.2, U15.3, led7.2 (A)
- new net D6_24V: R13.2, U16.1
- new net D7: A1.D7, R16.2
- new net D7_24V: R18.2, U11.4, U17.3, led8.2 (A)
- new net D8: A1.D8, R20.2
- new net D8_24V: R21.2, U11.3, U19.3, led9.2 (A)
- new net D9: A1.D9, R17.2
- new net D9_24V: R19.2, U11.2, U18.3, led10.2 (A)
- new net GNDA: K1.COM, K2.COM, K3.COM, R10.1, R11.1, R14.1, R15.1, R18.1, R19.1, R21.1, R22.2, R7.1, U9.1
Other:
- note added: "24v input"
- note added: "24v output"
- note added: "Relay"
- moved on the sheet: C1, C2, C3, H1, H2, H3, H4, J1, J3, J5, J6, J7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

Commit message: Add files via upload
Parts:
- removed A1: Arduino_Leonardo_pin_remove_2pin, hoshina_library:arduino_leonard_remove_2pin, symbol hoshina_library:Arduino_Leonardo_pin_remove_2pin
- removed T1, T2, T3: 2SD1781K, hoshina_library:2SD1781, symbol hoshina_library:2SD1781K
- removed U2, U3, U5: microB_usb_connector, hoshina_library:USB_Micro-B_MC5F-03_aitendo_reverse, symbol hoshina_library:microB_usb_connector
- removed U7: HDMI_Hole2, hoshina_library:HDMI_Hole2, symbol hoshina_library:HDMI_Hole2
- added A1: Arduino_Leonardo_pin_remove_4pin, hoshina_library:arduino_leonard_remove_4pin, symbol hoshina_library:Arduino_Leonardo_pin_remove_4pin
- added J10, J11, J13: USB_B_Micro, hoshina_library:USB_Micro-B_Molex_47346-0001, symbol Connector:USB_B_Micro
- added R33, R34, R35, R36, R37, R38, R39, R40, R41, R42: R, hoshina_library:carbon_register_1_6W_, symbol Device:R
- added R43, R44: 200/0.06W_chip, hoshina_library:register_0603, symbol Device:R
- added RA1: YC324J-10KCT-ND, hoshina_library:YC324J-10KCT-ND, symbol hoshina_library:YC324J-10KCT-ND
- added T1, T2, T3: S9013_trangister_elecrow, hoshina_library:S9013, symbol hoshina_library:S9013_trangister_elecrow
- added U4: aray_register_10k(1/8W), hoshina_library:array_register, symbol hoshina_library:aray_register
- C1, C2, C3: footprint hoshina_library:CP_EIA-2012-12_Kemet-R_Pad1.30x1.05mm_HandSolder -> hoshina_library:capa1608
- R1: value R -> 2.7k_chip
- R10, R11, R14, R15: value 10k -> 10k/0.0025W
- R16, R20: value 190 -> 200/0.06W_chip
- R17, R6: value 190 -> R; footprint hoshina_library:register_0603 -> hoshina_library:carbon_register_1_6W_
- R18, R19, R21, R7: value 10k -> R; footprint hoshina_library:register_0603 -> hoshina_library:carbon_register_1_6W_
- R2, R23, R24, R29, R30, R31, R32: value 5.6k/1w -> 4.7k/1w
- R22: value R -> 3.1k/1W
- R25, R26, R27, R28: value 4.7k -> 4.7k/0.06W
- R3, R4, R5: value 5k -> 5.1k/0.005W
- hand_electric_line1: footprint hoshina_library:2pin_power_gnd -> hoshina_library:XH2_pin
Connections:
- net +5V: now also J10.1 (VBUS), J11.1 (VBUS), J13.1 (VBUS)
- net A0: now also A1.A0
- net A1: now also A1.A1
- net A2: now also A1.A2
- net A3: now also A1.A3
- net D10: now also A1.D10, R38.1, R44.2; no longer R6.2
- net D10_24V: now also RA1.4, U4.4; no longer R7.2
- net D11: now also A1.D11, R39.2
- net D12: now also A1.D12, R40.2
- net D13: now also A1.D13, R41.2
- net D3: now also R6.2, A1.D3/SCL
- net D4: now also R17.2, A1.D4
- net D5: now also R7.2, A1.D5
- net D6: now also R18.2, A1.D6
- net D7: now also A1.D7, R35.1
- net D7_24V: now also RA1.1, U4.1; no longer R18.2
- net D8: now also A1.D8, R37.1, R43.2; no longer R20.2
- net D8_24V: now also RA1.2, U4.2; no longer R21.2
- net D9: now also R20.2, A1.D9, R36.1; no longer R17.2
- net D9_24V: now also RA1.3, U4.3; no longer R19.2
- net GND: now also R19.1, R21.1, A1.GND, J10.5 (GND), J11.5 (GND), J13.5 (GND), R33.1, R34.1, R42.1, T1.E, T2.E, T3.E
- net GNDA: now also R17.1, R6.1, RA1.5, RA1.6, RA1.7, RA1.8, U4.com; no longer R19.1, R21.1
- net at U1.DMU: now also J13.2 (D-)
- net at U1.DPU: now also J13.3 (D+)
- net at R1.2, U1.REXT: now also R42.2
- net at SW1.3: now also A1.RESET
- net at K1.C2, U20.2: now also T1.C
- net at K2.C2, U21.2: now also T2.C
- net at K3.C2, U22.2: now also T3.C
- net at R3.1: now also R39.1, T1.B
- net at J4.3 (D+): now also J11.3 (D+)
- net at J4.2 (D-): now also J11.2 (D-)
- net at R4.1: now also R40.1, T2.B
- net at R5.1: now also R41.1, T3.B
- net at J2.3 (D+): now also J10.3 (D+)
- net at J2.2 (D-): now also J10.2 (D-)
- net at U10.1: now also R38.2, R44.1; no longer R6.1
- net at R20.1: now also U18.1, R36.2; no longer U19.1
- net at R16.1, U17.1: now also R35.2
- net at R25.1, led4.1 (K): now also R19.2
- net at R26.1, led5.1 (K): now also R21.2
- net at R27.1, led6.1 (K): now also R33.2
- net at R28.1, led7.1 (K): now also R34.2
- new net: R37.2, R43.1, U19.1
Other:
- moved on the sheet: R1, R10, R11, R14, R15, R16, R25, R26, R27, R28, led4, led5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
