File: dobot_circuite/dobot_circuite.kicad_pcb (KiCad board)
At the start: 2 copper layers, 146 x 146 mm, 29 parts, among them J1 USB_A, J2 USB_A, J3 USB_A, J4 USB_A, J5 USB_A, J6 USB_A, J7 HDMI, J8 Jack-DC, J9 HDMI, U1 FE1.1s, U2 FE1.1s, U3 usb_connector, U4 XH_DCJ, U5 usb_connector, U6 HDMI_Hole, U7 HDMI_Hole2, U8 arduino_leonard, Y1 Crystal, Y2 Crystal

Commit message: Add files via upload
Parts:
- removed U4: XH_DCJ, hoshina_library:S2B-XH-A_DCJ
- removed U6: HDMI_Hole, hoshina_library:HDMI_Hole
- removed Y2: Crystal, hoshina_library:Crystal_SMD_5032-2Pin_5.0x3.2mm
- added A1: Arduino_Leonardo_pin_remove_2pin, hoshina_library:arduino_leonard_remove_2pin, F.Cu at (110.5, -125.7)
- added D1: LED_green, hoshina_library:LED_1608, F.Cu at (148.7, -33.5)
- added K1: ALQ105, hoshina_library:ALQ105_akituki, F.Cu at (126.1, -46.2)
- added K2: ALQ105, hoshina_library:ALQ105_akituki, F.Cu at (112.8, -46.2)
- added K3: ALQ105, hoshina_library:ALQ105_akituki, F.Cu at (100.1, -46.2)
- added R10: 10k, hoshina_library:register_0603, B.Cu at (49.9, -94.5)
- added R11: 10k, hoshina_library:register_0603, B.Cu at (60.5, -94.1)
- added R12: 1k/1W, hoshina_library:carbon_register, B.Cu at (52.7, -85.1)
- added R13: 1k/1W, hoshina_library:carbon_register, B.Cu at (73.7, -84.7)
- added R14: 10k, hoshina_library:register_0603, B.Cu at (38.0, -94.5)
- added R15: 10k, hoshina_library:register_0603, B.Cu at (70.6, -94.1)
- added R16: 190, hoshina_library:register_0603, B.Cu at (68.1, -31.4)
- added R17: 190, hoshina_library:register_0603, B.Cu at (51.8, -35.3)
- added R18: 10k, hoshina_library:register_0603, B.Cu at (68.1, -42.7)
- added R19: 10k, hoshina_library:register_0603, B.Cu at (51.8, -39.8)
- added R20: 190, hoshina_library:register_0603, B.Cu at (63.0, -33.9)
- added R21: 10k, hoshina_library:register_0603, B.Cu at (63.0, -40.5)
- added R22: R, hoshina_library:carbon_register, F.Cu at (133.5, -30.1)
- added R23: 5.6k/1w, hoshina_library:carbon_register, F.Cu at (133.5, -60.4)
- added R24: 5.6k/1w, hoshina_library:carbon_register, F.Cu at (133.5, -70.5)
- added R25: 4.7k, hoshina_library:register_0603, F.Cu at (7.03, -75.3)
- added R26: 4.7k, hoshina_library:register_0603, F.Cu at (7.03, -69.6)
- added R27: 4.7k, hoshina_library:register_0603, F.Cu at (7.03, -80.3)
- added R28: 4.7k, hoshina_library:register_0603, F.Cu at (7.03, -85.3)
- added R29: 5.6k/1w, hoshina_library:carbon_register, B.Cu at (26.0, -46.9)
- added R3: 5k, hoshina_library:register_0603, F.Cu at (126.1, -51.3)
- added R30: 5.6k/1w, hoshina_library:carbon_register, B.Cu at (26.1, -52.0)
- added R31: 5.6k/1w, hoshina_library:carbon_register, B.Cu at (25.9, -57.3)
- added R32: 5.6k/1w, hoshina_library:carbon_register, B.Cu at (25.9, -62.5)
- added R4: 5k, hoshina_library:register_0603, F.Cu at (112.8, -51.3)
- added R5: 5k, hoshina_library:register_0603, F.Cu at (100.1, -51.3)
- added R6: 190, hoshina_library:register_0603, B.Cu at (43.3, -34.7)
- added R7: 10k, hoshina_library:register_0603, B.Cu at (43.3, -39.8)
- added R8: 1k/1W, hoshina_library:carbon_register, B.Cu at (42.4, -86.0)
- added R9: 1k/1W, hoshina_library:carbon_register, B.Cu at (63.2, -84.7)
- added SW1: SW_Push_Dual, hoshina_library:SW_TH_Tactile_Omron_B3F-10xx, F.Cu at (4.83, -39.2)
- added T1: 2SD1781K, hoshina_library:2SD1781, F.Cu at (122.3, -51.9)
- added T2: 2SD1781K, hoshina_library:2SD1781, F.Cu at (109.0, -51.9)
- added T3: 2SD1781K, hoshina_library:2SD1781, F.Cu at (96.3, -51.9)
- added U10: fhoto_capura_PS817, hoshina_library:fhoto_capra_PS817, B.Cu at (41.4, -33.4)
- added U11: terminal_block_4pin_small, hoshina_library:terminal_block_4pin_small, F.Cu at (12.4, -62.6)
- added U12: fhoto_capura_PS817, hoshina_library:fhoto_capra_PS817, B.Cu at (50.4, -85.0)
- added U13: fhoto_capura_PS817, hoshina_library:fhoto_capra_PS817, B.Cu at (60.8, -84.7)
- added U14: fhoto_capura_PS817, hoshina_library:fhoto_capra_PS817, B.Cu at (38.4, -85.0)
- added U15: fhoto_capura_PS817, hoshina_library:fhoto_capra_PS817, B.Cu at (71.1, -84.7)
- added U16: terminal_block_4pin_small, hoshina_library:terminal_block_4pin_small, F.Cu at (12.4, -87.1)
- added U17: fhoto_capura_PS817, hoshina_library:fhoto_capra_PS817, B.Cu at (68.6, -33.3)
- added U18: fhoto_capura_PS817, hoshina_library:fhoto_capra_PS817, B.Cu at (49.9, -33.7)
- added U19: fhoto_capura_PS817, hoshina_library:fhoto_capra_PS817, B.Cu at (59.9, -33.0)
- added U20: diode_GS1010FL, hoshina_library:diode_GS1010FL, F.Cu at (122.3, -48.8)
- added U21: diode_GS1010FL, hoshina_library:diode_GS1010FL, F.Cu at (109.0, -48.8)
- added U22: diode_GS1010FL, hoshina_library:diode_GS1010FL, F.Cu at (96.3, -48.8)
- added U23: terminal_block_6pin_small, hoshina_library:terminal_block_6pin_small, F.Cu at (11.9, -121.6)
- added U9: terminal_block_2pin_small, hoshina_library:terminal_block_2pin_small, F.Cu at (139.4, -33.5)
- added hand_electric_line1: hoshina_library_terminal_block_2pin_small, hoshina_library:2pin_power_gnd, F.Cu at (76.2, -41.3)
- added led1: LED, hoshina_library:LED_1608, F.Cu at (148.7, -46.1)
- added led10: LED, hoshina_library:LED_1608, F.Cu at (6.67, -56.8)
- added led11: LED, hoshina_library:LED_1608, F.Cu at (6.67, -61.7)
- added led2: LED, hoshina_library:LED_1608, F.Cu at (148.7, -56.3)
- added led3: LED, hoshina_library:LED_1608, F.Cu at (148.7, -66.4)
- added led4: LED, hoshina_library:LED_1608, F.Cu at (7.05, -76.8)
- added led5: LED, hoshina_library:LED_1608, F.Cu at (7.05, -71.4)
- added led6: LED, hoshina_library:LED_1608, F.Cu at (7.05, -81.7)
- added led7: LED, hoshina_library:LED_1608, F.Cu at (7.05, -86.8)
- added led8: LED, hoshina_library:LED_1608, F.Cu at (6.67, -46.6)
- added led9: LED, hoshina_library:LED_1608, F.Cu at (6.67, -51.8)
- R2: value R -> 5.6k/1w; footprint hoshina_library:register_0603 -> hoshina_library:carbon_register
- U2: value FE1.1s -> microB_usb_connector; footprint hoshina_library:FE1.1s -> hoshina_library:USB_Micro-B_MC5F-03_aitendo_reverse
- U3, U5: value usb_connector -> microB_usb_connector; footprint hoshina_library:XH4PIN_S -> hoshina_library:USB_Micro-B_MC5F-03_aitendo_reverse
- U8: value arduino_leonard -> terminal_block_6pin_small; footprint hoshina_library:arduino_leonard -> hoshina_library:terminal_block_6pin_small
- moved H1 179.6 mm to (132.0, -132.0)
- moved J1 152.0 mm to (40.6, -143.5), turned to 180 degrees
- moved H3 120.2 mm to (22.0, -22.0)
- moved H4 119.3 mm to (22.0, -132.0)
- moved R2 104.8 mm to (133.5, -50.4)
- moved C2 78.5 mm to (54.9, -25.4)
- moved C1 77.1 mm to (60.9, -22.6)
- moved C3 77.1 mm to (54.9, -22.6)
- moved Y1 77.1 mm to (49.4, -16.5)
- moved U1 76.7 mm to (61.6, -17.1)
- moved R1 76.0 mm to (63.5, -14.6)
- moved U3 51.3 mm to (53.8, -52.7), turned to 0 degrees
- moved U5 32.2 mm to (73.7, -52.7)
- moved U2 31.3 mm to (34.4, -52.7), turned to 0 degrees
- moved Thinker_board1 26.6 mm to (52.3, -29.5)
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Connections:
- R2 pad 1: GND -> Net-(R2-Pad1)
- R2 pad 2: Net-(R2-Pad2) -> D13_relay
Routing:
- net GND: track 12.1 -> 698.6 mm, vias 2 -> 3
- net GNDA: track 0.00 -> 213.1 mm, vias 0 -> 6
- net +24V: track 0.00 -> 196.3 mm, vias 0 -> 1
- net D5: track 0.00 -> 184.6 mm, vias 0 -> 1
- net A0: track 0.00 -> 172.9 mm
- net Net-(A1-PadRESET): track 0.00 -> 171.5 mm, vias 0 -> 1
- net D3: track 0.00 -> 168.0 mm, vias 0 -> 2
- net A3: track 0.00 -> 162.8 mm
- net D4: track 0.00 -> 155.4 mm, vias 0 -> 3
- net D6: track 0.00 -> 142.3 mm, vias 0 -> 2
- net A2: track 0.00 -> 141.7 mm, vias 0 -> 2
- net A1: track 0.00 -> 140.4 mm, vias 0 -> 2
- net Net-(J6-Pad3): track 131.6 -> 20.8 mm, vias 0 -> 1
- net Net-(J6-Pad2): track 130.1 -> 19.4 mm, vias 0 -> 1
- net +5V: track 449.9 -> 549.2 mm, vias 0 -> 3
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Other:
- board size 146 x 146 mm -> 152 x 152 mm
- net class Default: clearance 0.1 -> 0.2
- rule trace_clearance: 0.1 -> 0.2
- rule trace_min: 0.125 -> 0.16
- board text added: "24V"
- board text added: "5V"
- board text added: "A0"
- board text added: "A1"
- board text added: "A2"
- board text added: "A3"
- board text added: "AIN(0-5V)"
- board text added: "D10"
- board text added: "D11"
- board text added: "D12"
- board text added: "D13"
- board text added: "D3"
- board text added: "D4"
- board text added: "D5"
- board text added: "D6"
- board text added: "D7"
- board text added: "D8"
- board text added: "D9"
- board text added: "GND"
- board text added: "IN(24V)"
- board text added: "OUT(24V)"
- board text added: "R1+"
- board text added: "R1-"
- board text added: "R2+"
- board text added: "R2-"
- board text added: "R3+"
- board text added: "R3-"
- board text added: "Relay(0-3A)"
- board text added: "pwr"
- board text added: "reset"

Commit message: Add files via upload
Parts:
- removed U2, U3, U5: microB_usb_connector, hoshina_library:USB_Micro-B_MC5F-03_aitendo_reverse
- removed U7: HDMI_Hole2, hoshina_library:HDMI_Hole2
- added J10: USB_B_Micro, hoshina_library:USB_Micro-B_Molex_47346-0001, B.Cu at (45.0, -60.0)
- added J11: USB_B_Micro, hoshina_library:USB_Micro-B_Molex_47346-0001, B.Cu at (60.0, -60.0)
- added J13: USB_B_Micro, hoshina_library:USB_Micro-B_Molex_47346-0001, B.Cu at (30.0, -60.0)
- added R33: R, hoshina_library:carbon_register_1_6W_, B.Cu at (40.6, -111.6)
- added R34: R, hoshina_library:carbon_register_1_6W_, B.Cu at (45.6, -111.6)
- added R35: R, hoshina_library:carbon_register_1_6W_, F.Cu at (53.3, -22.5)
- added R36: R, hoshina_library:carbon_register_1_6W_, F.Cu at (38.5, -22.5)
- added R37: R, hoshina_library:carbon_register_1_6W_, F.Cu at (45.9, -22.5)
- added R38: R, hoshina_library:carbon_register_1_6W_, F.Cu at (31.1, -22.5)
- added R39: R, hoshina_library:carbon_register_1_6W_, F.Cu at (117.5, -64.5)
- added R40: R, hoshina_library:carbon_register_1_6W_, F.Cu at (105.4, -64.5)
- added R41: R, hoshina_library:carbon_register_1_6W_, F.Cu at (93.2, -64.5)
- added R42: R, hoshina_library:carbon_register_1_6W_, F.Cu at (80.9, -22.5)
- added R43: 200/0.06W_chip, hoshina_library:register_0603, F.Cu at (43.8, -20.7)
- added R44: 200/0.06W_chip, hoshina_library:register_0603, F.Cu at (29.3, -20.7)
- added RA1: YC324J-10KCT-ND, hoshina_library:YC324J-10KCT-ND, F.Cu at (24.9, -40.9)
- added U4: aray_register_10k(1/8W), hoshina_library:array_register, B.Cu at (27.9, -36.8)
- A1: value Arduino_Leonardo_pin_remove_2pin -> Arduino_Leonardo_pin_remove_4pin; footprint hoshina_library:arduino_leonard_remove_2pin -> hoshina_library:arduino_leonard_remove_4pin
- C1, C2, C3: footprint hoshina_library:CP_EIA-2012-12_Kemet-R_Pad1.30x1.05mm_HandSolder -> hoshina_library:capa1608
- R1: value R -> 2.7k_chip
- R10, R11, R14, R15: value 10k -> 10k/0.0025W; moved to F.Cu
- R16, R20: value 190 -> 200/0.06W_chip; moved to F.Cu
- R17, R6: value 190 -> R; footprint hoshina_library:register_0603 -> hoshina_library:carbon_register_1_6W_; moved to F.Cu
- R18, R7: value 10k -> R; footprint hoshina_library:register_0603 -> hoshina_library:carbon_register_1_6W_; moved to F.Cu
- R19, R21: value 10k -> R; footprint hoshina_library:register_0603 -> hoshina_library:carbon_register_1_6W_
- R2, R23, R24, R29, R30, R31, R32: value 5.6k/1w -> 4.7k/1w
- R22: value R -> 3.1k/1W
- R25, R26, R27, R28: value 4.7k -> 4.7k/0.06W; moved to B.Cu
- R3, R4, R5: value 5k -> 5.1k/0.005W
- T1, T2, T3: value 2SD1781K -> S9013_trangister_elecrow; footprint hoshina_library:2SD1781 -> hoshina_library:S9013
- hand_electric_line1: footprint hoshina_library:2pin_power_gnd -> hoshina_library:XH2_pin
- moved J1 138.0 mm to (84.0, -12.5), turned to 0 degrees
- moved J3 131.4 mm to (40.0, -141.5), turned to 180 degrees
- moved R6 110.3 mm to (139.8, -88.1), turned to 270 degrees
- moved R7 100.1 mm to (130.9, -88.1), turned to 270 degrees
- moved R17 98.9 mm to (135.4, -88.1), turned to 270 degrees
- moved R14 95.3 mm to (133.1, -88.0), turned to 270 degrees
- moved R10 87.9 mm to (137.5, -88.0), turned to 270 degrees
- moved R21 78.3 mm to (30.4, -111.6), turned to 270 degrees
- moved R18 74.0 mm to (126.4, -88.3), turned to 270 degrees
- moved R19 73.7 mm to (35.4, -111.6)
- moved R11 68.5 mm to (128.7, -88.0), turned to 270 degrees
- moved R15 53.9 mm to (124.2, -88.0), turned to 270 degrees
- moved R26 48.7 mm to (28.3, -113.4), turned to 90 degrees
- moved R25 46.3 mm to (33.4, -113.4), turned to 90 degrees
- moved R28 46.1 mm to (43.6, -113.4), turned to 90 degrees
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Connections:
- R17 pad 1: Net-(R17-Pad1) -> GNDA
- R17 pad 2: D9 -> D4
- R18 pad 2: D7_24V -> D6
- R19 pad 1: GNDA -> GND
- R19 pad 2: D9_24V -> Net-(R19-Pad2)
- R20 pad 2: D8 -> D9
- R21 pad 1: GNDA -> GND
- R21 pad 2: D8_24V -> Net-(R21-Pad2)
- R25 pad 1: Net-(R25-Pad1) -> Net-(R19-Pad2)
- R26 pad 1: Net-(R26-Pad1) -> Net-(R21-Pad2)
- R6 pad 1: Net-(R6-Pad1) -> GNDA
- R6 pad 2: D10 -> D3
- R7 pad 2: D10_24V -> D5
- U10 pad 1: Net-(R6-Pad1) -> Net-(R38-Pad2)
- U18 pad 1: Net-(R17-Pad1) -> Net-(R20-Pad1)
- U19 pad 1: Net-(R20-Pad1) -> Net-(R37-Pad2)
- led4 pad 1: Net-(R25-Pad1) -> Net-(R19-Pad2)
- led5 pad 1: Net-(R26-Pad1) -> Net-(R21-Pad2)
Routing:
- net GND: track 698.6 -> 0.00 mm, vias 3 -> 0
- net +5V: track 549.2 -> 347.3 mm, vias 3 -> 1
- net D5: track 184.6 -> 0.00 mm, vias 1 -> 0
- net A0: track 172.9 -> 0.00 mm
- net Net-(A1-PadRESET): track 171.5 -> 0.00 mm, vias 1 -> 0
- net D3: track 168.0 -> 0.00 mm, vias 2 -> 0
- net A3: track 162.8 -> 0.00 mm
- net D4: track 155.4 -> 0.00 mm, vias 3 -> 0
- net D6: track 142.3 -> 0.00 mm, vias 2 -> 0
- net A2: track 141.7 -> 0.00 mm, vias 2 -> 0
- net A1: track 140.4 -> 0.00 mm, vias 2 -> 0
- net Net-(J1-Pad3): track 139.4 -> 0.00 mm, vias 1 -> 0
- net Net-(J1-Pad2): track 137.9 -> 0.00 mm, vias 1 -> 0
- net Net-(J11-Pad3): track 106.8 -> 0.00 mm
- net +24V: track 196.3 -> 89.8 mm, vias 1 -> 0
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- removed copper zone on B.Cu, net GND
- removed copper zone on F.Cu, net GND
Other:
- outline, holes or cut-outs redrawn
- board text added: "10kΩ(1/6W)"
- board text added: "2.7kΩ(1/6W)"
- board text added: "200Ω(1/6W)"
- board text added: "4.7kΩ(1/6W)"
- board text added: "5.1kΩ(1/6W)"
- board text added: "SMD or Through-hole"
- board text added: "VCC"
- board text added: "camera1"
- board text added: "camera2"
- board text added: "dobot"

Commit message: Add files via upload
Changed lines of the file:
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@@
     (47 F.CrtYd user)
     (48 B.Fab user)
-    (49 F.Fab user hide)
+    (49 F.Fab user)
   )
   (setup
@@
       (effects (font (size 1 1) (thickness 0.15)))
     )
-    (fp_text value 10k/0.0025W (at -15.875 0.635 270) (layer F.Fab)
+    (fp_text value 10k/0.0025W (at -16.383 0.635 270) (layer F.Fab)
       (effects (font (size 1 1) (thickness 0.15)))
     )
@@
   (gr_line (start 33.147 -42.545) (end 52.197 -42.545) (layer B.SilkS) (width 0.12))
   (gr_line (start 33.147 -52.07) (end 33.147 -42.545) (layer B.SilkS) (width 0.12))
-  (gr_text "SMD or Through-hole" (at 85.217 -18.034) (layer F.SilkS)
+  (gr_text "SMD or Through-hole" (at 85.217 -18.034) (layer F.Fab)
     (effects (font (size 1 1) (thickness 0.15) italic))
   )
@@
     (effects (font (size 1 1) (thickness 0.15)))
   )
-  (gr_text "SMD or Through-hole" (at 49.276 -24.892) (layer F.SilkS)
+  (gr_text "SMD or Through-hole" (at 49.276 -24.892) (layer F.Fab)
     (effects (font (size 1 1) (thickness 0.15) italic))
   )
@@
   (gr_line (start 121.285 -66.421) (end 121.285 -61.341) (layer F.SilkS) (width 0.12))
   (gr_line (start 89.535 -66.421) (end 121.285 -66.421) (layer F.SilkS) (width 0.12))
-  (gr_text "SMD or Through-hole" (at 131.191 -82.931) (layer F.SilkS)
+  (gr_text "SMD or Through-hole" (at 131.191 -82.931) (layer F.Fab)
     (effects (font (size 1 1) (thickness 0.15) italic))
   )
