File: thinker_board_shield_xhconnector/thinker_board_shield.kicad_pcb (KiCad board)
At the start: 4 copper layers, 56 x 65 mm, 5 parts, among them J1 Jack-DC, J2 Thinker_board_S

Commit message: Add files via upload
Parts:
- removed J1: Jack-DC, hoshina_library:DCJ
- added U1: XH_S, hoshina_library:S2B-XH-A, B.Cu at (13.0, 13.0)
- moved H1 75.9 mm to (3.50, 3.50)
- moved H3 75.9 mm to (52.5, 61.5)
Routing:
- net GND: track 93.3 -> 83.4 mm
Other:
- board text added: "GND"
- board text added: "VCC"
