File: thinker_board_shield_xhconnector/thinker_board_shield.sch (KiCad schematic (older format))
At the start: 5 parts, among them J1 Jack-DC, J2 Thinker_board_S

Commit message: Add files via upload
Parts:
- removed H? (x3): Hole_2.7mm, symbol hoshina_library:Hole_2.7mm
- removed J1: Jack-DC, hoshina_library:DCJ, symbol Connector:Jack-DC
- added H1, H2, H3: Hole_2.7mm, hoshina_library:Hole_2.7mm, symbol hoshina_library:Hole_2.7mm
- added U1: XH_S, hoshina_library:S2B-XH-A, symbol hoshina_library:XH_S
Connections:
- wire segments 19 -> 21
Changed lines of the file:
@@
 	1    0    0    -1
 $EndComp
-$Comp
-L Connector:Jack-DC J1
-U 1 1 5D71DF43
-P 2450 3500
-F 0 "J1" H 2507 3825 50  0000 C CNN
-F 1 "Jack-DC" H 2507 3734 50  0000 C CNN
-F 2 "hoshina_library:DCJ" H 2500 3460 50  0001 C CNN
-F 3 "~" H 2500 3460 50  0001 C CNN
-	1    2450 3500
-	1    0    0    -1
-$EndComp
-Text GLabel 2750 3400 2    50   Input ~ 0
+Text GLabel 2700 3500 2    50   Input ~ 0
 5V
-Text GLabel 2750 3600 2    50   Input ~ 0
+Text GLabel 2700 3400 2    50   Input ~ 0
 GND
 Text GLabel 4450 3000 0    50   Input ~ 0
@@
 	5000 5900 5000 5800
 Connection ~ 4900 5900
+Wire Wire Line
+	2600 3400 2700 3400
+Wire Wire Line
+	2700 3500 2600 3500
 $Comp
-L hoshina_library:Hole_2.7mm H?
-U 1 1 5D70F57A
-P 2650 2700
-F 0 "H?" H 2728 2746 50  0000 L CNN
-F 1 "Hole_2.7mm" H 2728 2655 50  0000 L CNN
-F 2 "" H 2650 2550 50  0001 C CNN
-F 3 "" H 2650 2550 50  0001 C CNN
-	1    2650 2700
+L hoshina_library:XH_S U1
+U 1 1 5D710EE3
+P 2600 3400
+F 0 "U1" H 2643 3219 50  0000 C CNN
+F 1 "XH_S" H 2643 3310 50  0000 C CNN
+F 2 "hoshina_library:S2B-XH-A" H 2600 3300 50  0001 C CNN
+F 3 "" H 2600 3300 50  0001 C CNN
+	1    2600 3400
+	-1   0    0    1
+$EndComp
+$Comp
+L hoshina_library:Hole_2.7mm H1
+U 1 1 5D712F7D
+P 2550 2250
+F 0 "H1" H 2628 2296 50  0000 L CNN
+F 1 "Hole_2.7mm" H 2628 2205 50  0000 L CNN
+F 2 "hoshina_library:Hole_2.7mm" H 2550 2100 50  0001 C CNN
+F 3 "" H 2550 2100 50  0001 C CNN
+	1    2550 2250
 	1    0    0    -1
 $EndComp
 $Comp
-L hoshina_library:Hole_2.7mm H?
-U 1 1 5D70F74E
-P 2650 2900
-F 0 "H?" H 2728 2946 50  0000 L CNN
-F 1 "Hole_2.7mm" H 2728 2855 50  0000 L CNN
-F 2 "" H 2650 2750 50  0001 C CNN
-F 3 "" H 2650 2750 50  0001 C CNN
-	1    2650 2900
+L hoshina_library:Hole_2.7mm H2
+U 1 1 5D712FF0
+P 2550 2500
+F 0 "H2" H 2628 2546 50  0000 L CNN
+F 1 "Hole_2.7mm" H 2628 2455 50  0000 L CNN
+F 2 "hoshina_library:Hole_2.7mm" H 2550 2350 50  0001 C CNN
+F 3 "" H 2550 2350 50  0001 C CNN
+	1    2550 2500
 	1    0    0    -1
 $EndComp
 $Comp
-L hoshina_library:Hole_2.7mm H?
-U 1 1 5D70FA54
-P 2650 2500
-F 0 "H?" H 2728 2546 50  0000 L CNN
-F 1 "Hole_2.7mm" H 2728 2455 50  0000 L CNN
-F 2 "" H 2650 2350 50  0001 C CNN
-F 3 "" H 2650 2350 50  0001 C CNN
-	1    2650 2500
+L hoshina_library:Hole_2.7mm H3
+U 1 1 5D7131FF
+P 2550 2750
+F 0 "H3" H 2628 2796 50  0000 L CNN
+F 1 "Hole_2.7mm" H 2628 2705 50  0000 L CNN
+F 2 "hoshina_library:Hole_2.7mm" H 2550 2600 50  0001 C CNN
+F 3 "" H 2550 2600 50  0001 C CNN
+	1    2550 2750
 	1    0    0    -1
 $EndComp
